Commit message: factory v1.1

File: model/factory.urdf.xacro (robot description, xacro)
@@ -5,4 +5,5 @@
   <xacro:include filename="$(find vito_description)/model/table.urdf.xacro"/>
   <xacro:include filename="$(find dual_manipulation_shared)/model/shelf.urdf.xacro"/>
+  <xacro:include filename="$(find dual_manipulation_shared)/model/conveyor_belt.urdf.xacro"/>
   <xacro:include filename="$(find vito_description)/model/materials.urdf"/>
   <xacro:include filename="$(find lwr_description)/model/kuka_lwr.urdf.xacro"/>
@@ -53,5 +54,5 @@
     <origin xyz="2.0 0 0" rpy="0 0 0"/>
   </xacro:model_table>
-    <xacro:model_table name="table3"
+<!--    <xacro:model_table name="table3"
                     parent="world"
                     length="1.0"
@@ -68,5 +69,13 @@
                     plate_thickness="0.1">
     <origin xyz="5.0 0 0" rpy="0 0 0"/>
-  </xacro:model_table>
+  </xacro:model_table>-->
+    <xacro:model_belt name="belt0"
+                      parent="world"
+                      length="2"
+                      width="1.0"
+                      height="0.0"
+                      plate_thickness="0.05">
+    <origin xyz="3.5 0 0" rpy="0 0 0"/>
+    </xacro:model_belt>
     <xacro:model_table name="table5"
                     parent="world"
@@ -114,12 +123,12 @@
   </xacro:soft_hand>
   <!-- LEFT ARM 2 -->
-  <xacro:kuka_lwr name="left_arm_2" parent="world">
+<!--  <xacro:kuka_lwr name="left_arm_2" parent="world">
     <origin xyz="4.5 0.2 0.60"
       rpy="${M_PI*80/180} ${M_PI*180.0/180} ${M_PI*0.0/180}"/>
-  </xacro:kuka_lwr>
-  <!-- LEFT SOFTHAND 1 -->
-  <xacro:soft_hand parent="left_arm_2_7_link" name="left_hand_2" left="true" withAdaptiveTransmission="true" useMimicTag="true">
+  </xacro:kuka_lwr>-->
+  <!-- LEFT SOFTHAND 2 -->
+<!--  <xacro:soft_hand parent="left_arm_2_7_link" name="left_hand_2" left="true" withAdaptiveTransmission="true" useMimicTag="true">
     <origin xyz="0 0 0" rpy="0 0 0"/>
-  </xacro:soft_hand>
+  </xacro:soft_hand>-->
   <!-- RIGHT ARM 2 -->
   <xacro:kuka_lwr name="right_arm_2" parent="world">
@@ -127,5 +136,5 @@
       rpy="${M_PI*-80/180} ${M_PI*180.0/180} ${M_PI*0.0/180}"/>
   </xacro:kuka_lwr>
-  <!-- RIGHT SOFTHAND 1 -->
+  <!-- RIGHT SOFTHAND 2 -->
   <xacro:soft_hand parent="right_arm_2_7_link" name="right_hand_2" left="false" withAdaptiveTransmission="true" useMimicTag="true">
     <origin xyz="0 0 0" rpy="0 0 0"/>

Commit message: changed factory xacro to have an anchor link

File: model/factory.urdf.xacro (robot description, xacro)
@@ -9,8 +9,13 @@
   <xacro:include filename="$(find lwr_description)/model/kuka_lwr.urdf.xacro"/>
   <xacro:include filename="$(find soft_hand_description)/model/soft_hand.urdf.xacro"/>
-  <link name="world" />
+  <!-- <link name="world" />
+  <joint name="factory_world_joint" type="fixed">
+    <parent link="world" />
+    <child link="factory_anchor" />
+  </joint> -->
+  <link name="factory_anchor" />
   <!-- MISC -->
   <xacro:model_shelf name="shelf0"
-                    parent="world"
+                    parent="factory_anchor"
                     length="0.1"
                     width="1.30"
@@ -21,5 +26,5 @@
   </xacro:model_shelf>
   <xacro:model_shelf name="shelf1"
-                    parent="world"
+                    parent="factory_anchor"
                     length="0.4"
                     width="1.30"
@@ -31,5 +36,5 @@
   <!-- TABLES -->
   <xacro:model_table name="table0"
-                    parent="world"
+                    parent="factory_anchor"
                     length="1.0"
                     width="1.30"
@@ -39,5 +44,5 @@
   </xacro:model_table>
     <xacro:model_table name="table1"
-                    parent="world"
+                    parent="factory_anchor"
                     length="1.0"
                     width="1.30"
@@ -47,5 +52,5 @@
   </xacro:model_table>
     <xacro:model_table name="table2"
-                    parent="world"
+                    parent="factory_anchor"
                     length="0.8"
                     width="1.30"
@@ -55,5 +60,5 @@
   </xacro:model_table>
 <!--    <xacro:model_table name="table3"
-                    parent="world"
+                    parent="factory_anchor"
                     length="1.0"
                     width="1.30"
@@ -63,5 +68,5 @@
   </xacro:model_table>
     <xacro:model_table name="table4"
-                    parent="world"
+                    parent="factory_anchor"
                     length="1.0"
                     width="1.30"
@@ -71,5 +76,5 @@
   </xacro:model_table>-->
     <xacro:model_belt name="belt0"
-                      parent="world"
+                      parent="factory_anchor"
                       length="2"
                       width="1.0"
@@ -79,5 +84,5 @@
     </xacro:model_belt>
     <xacro:model_table name="table5"
-                    parent="world"
+                    parent="factory_anchor"
                     length="1.0"
                     width="1.30"
@@ -87,5 +92,5 @@
   </xacro:model_table>
   <!-- LEFT ARM 0 -->
-  <xacro:kuka_lwr name="0_left_arm" parent="world">
+  <xacro:kuka_lwr name="0_left_arm" parent="factory_anchor">
     <origin xyz="0.5 0.2 0.60"
       rpy="${M_PI*80/180} ${M_PI*180.0/180} ${M_PI*0.0/180}"/>
@@ -96,5 +101,5 @@
   </xacro:soft_hand>
   <!-- RIGHT ARM 0 -->
-  <xacro:kuka_lwr name="0_right_arm" parent="world">
+  <xacro:kuka_lwr name="0_right_arm" parent="factory_anchor">
     <origin xyz="1.5 -1.5 0.60"
       rpy="${M_PI*-80/180} ${M_PI*180.0/180} ${M_PI*0.0/180}"/>
@@ -105,5 +110,5 @@
   </xacro:soft_hand>
   <!-- LEFT ARM 1 -->
-  <xacro:kuka_lwr name="1_left_arm" parent="world">
+  <xacro:kuka_lwr name="1_left_arm" parent="factory_anchor">
     <origin xyz="2.5 0.2 0.60"
       rpy="${M_PI*80/180} ${M_PI*180.0/180} ${M_PI*0.0/180}"/>
@@ -114,5 +119,5 @@
   </xacro:soft_hand>
   <!-- RIGHT ARM 1 -->
-  <xacro:kuka_lwr name="1_right_arm" parent="world">
+  <xacro:kuka_lwr name="1_right_arm" parent="factory_anchor">
     <origin xyz="3.5 -1.5 0.60"
       rpy="${M_PI*-80/180} ${M_PI*180.0/180} ${M_PI*0.0/180}"/>
@@ -123,5 +128,5 @@
   </xacro:soft_hand>
   <!-- LEFT ARM 2 -->
-<!--  <xacro:kuka_lwr name="2_left_arm" parent="world">
+<!--  <xacro:kuka_lwr name="2_left_arm" parent="factory_anchor">
     <origin xyz="4.5 0.2 0.60"
       rpy="${M_PI*80/180} ${M_PI*180.0/180} ${M_PI*0.0/180}"/>
@@ -132,5 +137,5 @@
   </xacro:soft_hand>-->
   <!-- RIGHT ARM 2 -->
-  <xacro:kuka_lwr name="2_right_arm" parent="world">
+  <xacro:kuka_lwr name="2_right_arm" parent="factory_anchor">
     <origin xyz="5.5 -1.5 0.60"
       rpy="${M_PI*-80/180} ${M_PI*180.0/180} ${M_PI*0.0/180}"/>

Commit message: changed origins to have tables at the same height

File: model/factory.urdf.xacro (robot description, xacro)
@@ -23,5 +23,5 @@
                     plate_thickness="0.4"
 		    color="Grey">
-    <origin xyz="1.0 0 0" rpy="0 0 0"/>
+    <origin xyz="1.0 0 0.07" rpy="0 0 0"/>
   </xacro:model_shelf>
   <xacro:model_shelf name="shelf1"
@@ -32,5 +32,5 @@
                     plate_thickness="0.1"
 		    color="DarkGrey">
-    <origin xyz="0.8 0 0" rpy="0 0 0"/>
+    <origin xyz="0.8 0 0.07" rpy="0 0 0"/>
   </xacro:model_shelf>
   <!-- TABLES -->
@@ -41,5 +41,5 @@
                     height="0.9"
                     plate_thickness="0.1">
-    <origin xyz="0 0 0" rpy="0 0 0"/>
+    <origin xyz="0 0 0.07" rpy="0 0 0"/>
   </xacro:model_table>
     <xacro:model_table name="table1"
@@ -49,5 +49,5 @@
                     height="0.9"
                     plate_thickness="0.1">
-    <origin xyz="1.0 0 0" rpy="0 0 0"/>
+    <origin xyz="1.0 0 0.07" rpy="0 0 0"/>
   </xacro:model_table>
     <xacro:model_table name="table2"
@@ -57,5 +57,5 @@
                     height="0.9"
                     plate_thickness="0.1">
-    <origin xyz="2.0 0 0" rpy="0 0 0"/>
+    <origin xyz="2.0 0 0.07" rpy="0 0 0"/>
   </xacro:model_table>
 <!--    <xacro:model_table name="table3"
@@ -90,5 +90,5 @@
                     height="0.9"
                     plate_thickness="0.1">
-    <origin xyz="6.0 0 0" rpy="0 0 0"/>
+    <origin xyz="6.0 0 0.07" rpy="0 0 0"/>
   </xacro:model_table>
   <!-- LEFT ARM 0 -->
