Commit message: fixed little issues

File: model/conveyor_belt.urdf.xacro (robot description, xacro)
@@ -1,4 +1,4 @@
 <?xml version="1.0"?>
-<robot xmlns:xacro="http://www.ros.org/wiki/xacro">
+<robot xmlns:xacro="http://www.ros.org/wiki/xacro" name="belt">
 <xacro:property name="border_offset" value="0.055" />
 <!-- conversions -->
@@ -87,5 +87,5 @@
     </link>
      <joint name="${name}_joint" type="prismatic">
-        <origin xyz="0.3 ${-1/2 * width} ${height+plate_thickness/2.0}"
+        <origin xyz="0.3 ${-1/2 * width} ${height+plate_thickness/2.0+0.01}"
             rpy="${M_PI*0.0/180} ${M_PI*0.0/180} ${M_PI*0.0/180}"/>
         <axis xyz="1 0 0"/>

Commit message: fixed wrong displacement

File: model/conveyor_belt.urdf.xacro (robot description, xacro)
@@ -25,5 +25,5 @@
         </inertial>
         <visual>
-            <origin xyz="${1/2 * length} ${-1/2 * width} ${height}"/>
+            <origin xyz="${1/2 * length} ${-1/2 * width-0.125} ${height}"/>
             <geometry>
                 <box size="${length} ${width} ${plate_thickness}"/>
@@ -32,5 +32,5 @@
 		</visual>
         <collision>
-            <origin xyz="${1/2 * length} ${-1/2 * width} ${height}"/>
+            <origin xyz="${1/2 * length} ${-1/2 * width-0.125} ${height}"/>
             <geometry>
                 <box size="${length} ${width} ${plate_thickness}"/>
@@ -47,5 +47,5 @@
         </inertial>
         <visual>
-            <origin xyz="0 ${-1/2 * width} ${height}"
+            <origin xyz="0 ${-1/2 * width-0.125} ${height}"
             rpy="${M_PI*90/180} ${M_PI*0.0/180} ${M_PI*0.0/180}"/>
             <geometry>
@@ -55,5 +55,5 @@
 		</visual>
         <collision>
-            <origin xyz="0 ${-1/2 * width} ${height}"
+            <origin xyz="0 ${-1/2 * width-0.125} ${height}"
             rpy="${M_PI*90/180} ${M_PI*0.0/180} ${M_PI*0.0/180}"/>
             <geometry>
@@ -71,5 +71,5 @@
         </inertial>
         <visual>
-            <origin xyz="${length} ${-1/2 * width} ${height}"
+            <origin xyz="${length} ${-1/2 * width-0.125} ${height}"
             rpy="${M_PI*90/180} ${M_PI*0.0/180} ${M_PI*0.0/180}"/>
             <geometry>
@@ -79,5 +79,5 @@
 		</visual>
         <collision>
-            <origin xyz="${length} ${-1/2 * width} ${height}"
+            <origin xyz="${length} ${-1/2 * width-0.125} ${height}"
             rpy="${M_PI*90/180} ${M_PI*0.0/180} ${M_PI*0.0/180}"/>
             <geometry>
@@ -87,5 +87,5 @@
     </link>
      <joint name="${name}_joint" type="prismatic">
-        <origin xyz="0.3 ${-1/2 * width} ${height+plate_thickness/2.0+0.01}"
+        <origin xyz="0.3 ${-1/2 * width-0.125} ${height+plate_thickness/2.0+0.01}"
             rpy="${M_PI*0.0/180} ${M_PI*0.0/180} ${M_PI*0.0/180}"/>
         <axis xyz="1 0 0"/>

Commit message: added a joint to get the belt to be considered as a chain

File: model/conveyor_belt.urdf.xacro (robot description, xacro)
@@ -93,4 +93,17 @@
         <dynamics friction="10.0" damping="1.0"/>
         <parent link="${name}_plate_link"/>
+        <child link="${name}_p_1"/>
+    </joint>
+    <link name="${name}_p_1">
+        <inertial>
+            <insert_block name="negligible_inertia"/>
+        </inertial>
+    </link>
+    <!-- This additional joint is needed for KDLKinematicsPlugin to work properly (it needs at least two active joints to consider this a chain!!!) -->
+    <joint name="${name}_joint_r1" type="revolute">
+        <origin xyz="0 0 0" rpy="0 0 0"/>
+        <axis xyz="0 0 1"/>
+        <limit lower="-0.001" upper="0.001" effort="200" velocity="10" />
+        <parent link="${name}_p_1"/>
         <child link="${name}_p"/>
     </joint>
@@ -106,5 +119,5 @@
             </geometry>
             <material name="Vito/Orange"/>
-	</visual>
+        </visual>
         <collision>
             <origin xyz="0 0 0"

File: model/factory.urdf.xacro (robot description, xacro)
@@ -20,6 +20,6 @@
                     length="0.1"
                     width="1.30"
-                    height="0.3"
-                    plate_thickness="0.3"
+                    height="0.4"
+                    plate_thickness="0.4"
 		    color="Grey">
     <origin xyz="1.0 0 0" rpy="0 0 0"/>
@@ -29,5 +29,5 @@
                     length="0.4"
                     width="1.30"
-                    height="0.4"
+                    height="0.5"
                     plate_thickness="0.1"
 		    color="DarkGrey">

Commit message: added legs to the conveyor belt

File: model/conveyor_belt.urdf.xacro (robot description, xacro)
@@ -14,5 +14,5 @@
     <inertia ixx="${negligible_mass * 10 * mm2_to_m2}" ixy="0.0" ixz="0.0" iyy="${negligible_mass * 10 * mm2_to_m2}" iyz="0.0" izz="${negligible_mass * 10 * mm2_to_m2}"/>
 </xacro:property>
-<xacro:macro name="model_belt" params="parent name *origin length width height plate_thickness">
+<xacro:macro name="model_belt" params="parent name *origin length width height leg_length plate_thickness">
     <joint name="${parent}_${name}_base_joint" type="fixed">
         <insert_block name="origin"/>
@@ -38,4 +38,5 @@
         </collision>
     </link>
+    <!-- TOP -->
     <joint name="${parent}_${name}_joint1" type="fixed">
         <parent link="${name}_plate_link"/>
@@ -50,5 +51,5 @@
             rpy="${M_PI*90/180} ${M_PI*0.0/180} ${M_PI*0.0/180}"/>
             <geometry>
-                <cylinder length="${width}" radius="${plate_thickness}"/>
+                <cylinder length="${width+0.01}" radius="${plate_thickness}"/>
 			</geometry>
 			<material name="Vito/Blue"/>
@@ -58,8 +59,57 @@
             rpy="${M_PI*90/180} ${M_PI*0.0/180} ${M_PI*0.0/180}"/>
             <geometry>
-                <cylinder length="${width}" radius="${plate_thickness}"/>
-            </geometry>
-        </collision>
-    </link>
+                <cylinder length="${width+0.01}" radius="${plate_thickness}"/>
+            </geometry>
+        </collision>
+    </link>
+    <joint name="${parent}_${name}_cylinder_joint1" type="fixed">
+        <parent link="${name}_link1"/>
+        <child link="${name}_cylinder_leg1"/>
+    </joint>
+    <link name="${name}_cylinder_leg1">
+        <inertial>
+            <insert_block name="negligible_inertia"/>
+        </inertial>
+        <visual>
+            <origin xyz="0 ${-1/5 * width -0.125} ${height-leg_length/2.0}"
+            rpy="${M_PI*0.0/180} ${M_PI*0.0/180} ${M_PI*0.0/180}"/>
+            <geometry>
+                <box size="0.05 0.05 ${leg_length}"/>
+			</geometry>
+			<material name="Vito/Black"/>
+		</visual>
+        <collision>
+            <origin xyz="0 ${-1/5 * width -0.125} ${height-leg_length/2.0}"
+            rpy="${M_PI*0.0/180} ${M_PI*0.0/180} ${M_PI*0.0/180}"/>
+            <geometry>
+                <box size="0.05 0.05 ${leg_length}"/>
+            </geometry>
+        </collision>
+    </link>
+    <joint name="${parent}_${name}_cylinder_joint2" type="fixed">
+        <parent link="${name}_link1"/>
+        <child link="${name}_cylinder_leg2"/>
+    </joint>
+    <link name="${name}_cylinder_leg2">
+        <inertial>
+            <insert_block name="negligible_inertia"/>
+        </inertial>
+        <visual>
+            <origin xyz="0 ${-4/5 * width -0.125} ${height-leg_length/2.0}"
+            rpy="${M_PI*0.0/180} ${M_PI*0.0/180} ${M_PI*0.0/180}"/>
+            <geometry>
+                <box size="0.05 0.05 ${leg_length}"/>
+			</geometry>
+			<material name="Vito/Black"/>
+		</visual>
+        <collision>
+            <origin xyz="0 ${-4/5 * width -0.125} ${height-leg_length/2.0}"
+            rpy="${M_PI*0.0/180} ${M_PI*0.0/180} ${M_PI*0.0/180}"/>
+            <geometry>
+                <box size="0.05 0.05 ${leg_length}"/>
+            </geometry>
+        </collision>
+    </link>
+    <!-- BOTTOM -->
     <joint name="${parent}_${name}_joint2" type="fixed">
         <parent link="${name}_plate_link"/>
@@ -74,5 +124,5 @@
             rpy="${M_PI*90/180} ${M_PI*0.0/180} ${M_PI*0.0/180}"/>
             <geometry>
-                <cylinder length="${width}" radius="${plate_thickness}"/>
+                <cylinder length="${width+0.01}" radius="${plate_thickness}"/>
 			</geometry>
 			<material name="Vito/Blue"/>
@@ -82,8 +132,57 @@
             rpy="${M_PI*90/180} ${M_PI*0.0/180} ${M_PI*0.0/180}"/>
             <geometry>
-                <cylinder length="${width}" radius="${plate_thickness}"/>
-            </geometry>
-        </collision>
-    </link>
+                <cylinder length="${width+0.01}" radius="${plate_thickness}"/>
+            </geometry>
+        </collision>
+    </link>
+    <joint name="${parent}_${name}_cylinder_joint3" type="fixed">
+        <parent link="${name}_link2"/>
+        <child link="${name}_cylinder_leg3"/>
+    </joint>
+    <link name="${name}_cylinder_leg3">
+        <inertial>
+            <insert_block name="negligible_inertia"/>
+        </inertial>
+        <visual>
+            <origin xyz="${length} ${-1/5 * width -0.125} ${height-leg_length/2.0}"
+            rpy="${M_PI*0.0/180} ${M_PI*0.0/180} ${M_PI*0.0/180}"/>
+            <geometry>
+                <box size="0.05 0.05 ${leg_length}"/>
+			</geometry>
+			<material name="Vito/Black"/>
+		</visual>
+        <collision>
+            <origin xyz="${length} ${-1/5 * width -0.125} ${height-leg_length/2.0}"
+            rpy="${M_PI*0.0/180} ${M_PI*0.0/180} ${M_PI*0.0/180}"/>
+            <geometry>
+                <box size="0.05 0.05 ${leg_length}"/>
+            </geometry>
+        </collision>
+    </link>
+    <joint name="${parent}_${name}_cylinder_joint4" type="fixed">
+        <parent link="${name}_link2"/>
+        <child link="${name}_cylinder_leg4"/>
+    </joint>
+    <link name="${name}_cylinder_leg4">
+        <inertial>
+            <insert_block name="negligible_inertia"/>
+        </inertial>
+        <visual>
+            <origin xyz="${length} ${-4/5 * width -0.125} ${height-leg_length/2.0}"
+            rpy="${M_PI*0.0/180} ${M_PI*0.0/180} ${M_PI*0.0/180}"/>
+            <geometry>
+                <box size="0.05 0.05 ${leg_length}"/>
+			</geometry>
+			<material name="Vito/Black"/>
+		</visual>
+        <collision>
+            <origin xyz="${length} ${-4/5 * width -0.125} ${height-leg_length/2.0}"
+            rpy="${M_PI*0.0/180} ${M_PI*0.0/180} ${M_PI*0.0/180}"/>
+            <geometry>
+                <box size="0.05 0.05 ${leg_length}"/>
+            </geometry>
+        </collision>
+    </link>
+    <!-- REAL ROBOT -->
      <joint name="${name}_joint" type="prismatic">
         <origin xyz="0.3 ${-1/2 * width-0.125} ${height+plate_thickness/2.0+0.01}"

File: model/factory.urdf.xacro (robot description, xacro)
@@ -80,4 +80,5 @@
                       width="1.0"
                       height="0.0"
+		      leg_length="0.9"
                       plate_thickness="0.05">
     <origin xyz="3.5 0 0" rpy="0 0 0"/>

Commit message: removed legs in the conveyor belt

File: model/conveyor_belt.urdf.xacro (robot description, xacro)
@@ -63,5 +63,5 @@
         </collision>
     </link>
-    <joint name="${parent}_${name}_cylinder_joint1" type="fixed">
+    <!-- <joint name="${parent}_${name}_cylinder_joint1" type="fixed">
         <parent link="${name}_link1"/>
         <child link="${name}_cylinder_leg1"/>
@@ -110,5 +110,5 @@
             </geometry>
         </collision>
-    </link>
+    </link> -->
     <!-- BOTTOM -->
     <joint name="${parent}_${name}_joint2" type="fixed">
@@ -136,5 +136,5 @@
         </collision>
     </link>
-    <joint name="${parent}_${name}_cylinder_joint3" type="fixed">
+   <!--  <joint name="${parent}_${name}_cylinder_joint3" type="fixed">
         <parent link="${name}_link2"/>
         <child link="${name}_cylinder_leg3"/>
@@ -183,5 +183,5 @@
             </geometry>
         </collision>
-    </link>
+    </link> -->
     <!-- REAL ROBOT -->
      <joint name="${name}_joint" type="prismatic">
