Commit message: took back tinoBot end-effector name

File: model/tinoBot.urdf.xacro (robot description, xacro)
@@ -96,9 +96,9 @@
       <origin xyz="0 0 0.025" rpy="0 0 0"/>
       <parent link="${name}_footprint"/>
-      <!-- <child link="${name}_ee"/> -->
-      <child link="belt0_p"/>
-    </joint>
-    <!-- <link name="${name}_ee"> -->
-    <link name="belt0_p">
+      <child link="${name}_ee"/>
+      <!-- <child link="belt0_p"/> -->
+    </joint>
+    <!-- <link name="belt0_p"> -->
+    <link name="${name}_ee">
       <visual>
         <origin xyz="0 0 0" rpy="0 0 0"/>

Commit message: added prefix to wheel links and limits as parameters in tinoBot

File: model/tinoBot.urdf.xacro (robot description, xacro)
@@ -33,9 +33,9 @@
   <property name="p_joint_effort" value="30"/>
   <property name="p_joint_velocity" value="10"/>
-  <property name="px_lower_limit" value="-2"/>
-  <property name="px_upper_limit" value="2"/>
-  <property name="py_lower_limit" value="-1"/>
-  <property name="py_upper_limit" value="1"/>
-  <xacro:macro name="tinoBot" params="parent name *origin">
+  <property name="px_lower_limit_def" value="-2"/>
+  <property name="px_upper_limit_def" value="2"/>
+  <property name="py_lower_limit_def" value="-1"/>
+  <property name="py_upper_limit_def" value="1"/>
+  <xacro:macro name="tinoBot" params="parent name *origin px_lower_limit:=${px_lower_limit_def} px_upper_limit:=${px_upper_limit_def} py_lower_limit:=${py_lower_limit_def} py_upper_limit:=${py_upper_limit_def}">
     <!-- <joint name="${name}_base_joint" type="fixed">
       <insert_block name="origin"/>
@@ -131,5 +131,5 @@
     </link>
     <!-- front left wheel -->
-    <joint name="caster_joint_fl" type="fixed"> <!-- type="continuous"> -->
+    <joint name="${name}_caster_joint_fl" type="fixed"> <!-- type="continuous"> -->
       <origin xyz="${caster_offset_x} ${caster_offset_y} ${caster_offset_z}" rpy="0 0 0"/>
       <!-- <axis xyz="0 0 1"/>
@@ -138,7 +138,7 @@
       <safety_controller k_velocity="${caster_joint_safety_k_velocity}"/> -->
       <parent link="${name}_link"/>
-      <child link="caster_link_fl"/>
-    </joint>
-    <link name="caster_link_fl">
+      <child link="${name}_caster_link_fl"/>
+    </joint>
+    <link name="${name}_caster_link_fl">
       <inertial>
         <mass value="${caster_mass}"/>
@@ -147,5 +147,5 @@
       </inertial>
     </link>
-    <joint name="wheel_joint_fl" type="fixed"> <!-- type="continuous"> -->
+    <joint name="${name}_wheel_joint_fl" type="fixed"> <!-- type="continuous"> -->
       <!-- <axis xyz="0 1 0"/>
       <limit effort="${wheel_joint_effort}" velocity="${wheel_joint_velocity}"/>
@@ -153,8 +153,8 @@
       <safety_controller k_velocity="${wheel_joint_safety_k_velocity}"/> -->
       <origin xyz="${wheel_offset_x} ${wheel_offset_y} ${wheel_offset_z}" rpy="0 0 0"/>
-      <parent link="caster_link_fl"/>
-      <child link="wheel_link_fl"/>
-    </joint>
-    <link name="wheel_link_fl">
+      <parent link="${name}_caster_link_fl"/>
+      <child link="${name}_wheel_link_fl"/>
+    </joint>
+    <link name="${name}_wheel_link_fl">
       <inertial>
         <mass value="${wheel_mass}"/>
@@ -178,5 +178,5 @@
     </link>
     <!-- front right wheel -->
-    <joint name="caster_joint_fr"  type="fixed"> <!-- type="continuous"> -->
+    <joint name="${name}_caster_joint_fr"  type="fixed"> <!-- type="continuous"> -->
       <origin xyz="${caster_offset_x} ${-caster_offset_y} ${caster_offset_z}" rpy="0 0 0"/>
       <!-- <axis xyz="0 0 1"/>
@@ -185,7 +185,7 @@
       <safety_controller k_velocity="${caster_joint_safety_k_velocity}"/> -->
       <parent link="${name}_link"/>
-      <child link="caster_link_fr"/>
-    </joint>
-    <link name="caster_link_fr">
+      <child link="${name}_caster_link_fr"/>
+    </joint>
+    <link name="${name}_caster_link_fr">
       <inertial>
         <mass value="${caster_mass}"/>
@@ -194,5 +194,5 @@
       </inertial>
     </link>
-    <joint name="wheel_joint_fr"  type="fixed"> <!-- type="continuous"> -->
+    <joint name="${name}_wheel_joint_fr"  type="fixed"> <!-- type="continuous"> -->
       <!-- <axis xyz="0 1 0"/>
       <limit effort="${wheel_joint_effort}" velocity="${wheel_joint_velocity}"/>
@@ -200,8 +200,8 @@
       <safety_controller k_velocity="${wheel_joint_safety_k_velocity}"/> -->
       <origin xyz="${wheel_offset_x} ${wheel_offset_y} ${wheel_offset_z}" rpy="0 0 0"/>
-      <parent link="caster_link_fr"/>
-      <child link="wheel_link_fr"/>
-    </joint>
-    <link name="wheel_link_fr">
+      <parent link="${name}_caster_link_fr"/>
+      <child link="${name}_wheel_link_fr"/>
+    </joint>
+    <link name="${name}_wheel_link_fr">
       <inertial>
         <mass value="${wheel_mass}"/>
@@ -225,5 +225,5 @@
     </link>
     <!-- back left wheel -->
-    <joint name="caster_joint_bl"  type="fixed"> <!-- type="continuous"> -->
+    <joint name="${name}_caster_joint_bl"  type="fixed"> <!-- type="continuous"> -->
       <origin xyz="${-caster_offset_x} ${caster_offset_y} ${caster_offset_z}" rpy="0 0 0"/>
       <!-- <axis xyz="0 0 1"/>
@@ -232,7 +232,7 @@
       <safety_controller k_velocity="${caster_joint_safety_k_velocity}"/> -->
       <parent link="${name}_link"/>
-      <child link="caster_link_bl"/>
-    </joint>
-    <link name="caster_link_bl">
+      <child link="${name}_caster_link_bl"/>
+    </joint>
+    <link name="${name}_caster_link_bl">
       <inertial>
         <mass value="${caster_mass}"/>
@@ -241,5 +241,5 @@
       </inertial>
     </link>
-    <joint name="wheel_joint_bl"  type="fixed"> <!-- type="continuous"> -->
+    <joint name="${name}_wheel_joint_bl"  type="fixed"> <!-- type="continuous"> -->
       <!-- <axis xyz="0 1 0"/>
       <limit effort="10" velocity="10"/>
@@ -248,8 +248,8 @@
       <safety_controller k_velocity="${wheel_joint_safety_k_velocity}"/> -->
       <origin xyz="${wheel_offset_x} ${wheel_offset_y} ${wheel_offset_z}" rpy="0 0 0"/>
-      <parent link="caster_link_bl"/>
-      <child link="wheel_link_bl"/>
-    </joint>
-    <link name="wheel_link_bl">
+      <parent link="${name}_caster_link_bl"/>
+      <child link="${name}_wheel_link_bl"/>
+    </joint>
+    <link name="${name}_wheel_link_bl">
       <inertial>
         <mass value="${wheel_mass}"/>
@@ -273,5 +273,5 @@
     </link>
     <!-- back right wheel -->
-    <joint name="caster_joint_br" type="fixed"> <!-- type="continuous"> -->
+    <joint name="${name}_caster_joint_br" type="fixed"> <!-- type="continuous"> -->
       <origin xyz="${-caster_offset_x} ${-caster_offset_y} ${caster_offset_z}" rpy="0 0 0"/>
       <!-- <axis xyz="0 0 1"/>
@@ -280,7 +280,7 @@
       <safety_controller k_velocity="${caster_joint_safety_k_velocity}"/> -->
       <parent link="${name}_link"/>
-      <child link="caster_link_br"/>
-    </joint>
-    <link name="caster_link_br">
+      <child link="${name}_caster_link_br"/>
+    </joint>
+    <link name="${name}_caster_link_br">
       <inertial>
         <mass value="${caster_mass}"/>
@@ -289,5 +289,5 @@
       </inertial>
     </link>
-    <joint name="wheel_joint_br" type="fixed"> <!-- type="continuous"> -->
+    <joint name="${name}_wheel_joint_br" type="fixed"> <!-- type="continuous"> -->
       <axis xyz="0 1 0"/>
       <!-- <limit effort="${wheel_joint_effort}" velocity="${wheel_joint_velocity}"/>
@@ -295,8 +295,8 @@
       <safety_controller k_velocity="${wheel_joint_safety_k_velocity}"/> -->
       <origin xyz="${wheel_offset_x} ${wheel_offset_y} ${wheel_offset_z}" rpy="0 0 0"/>
-      <parent link="caster_link_br"/>
-      <child link="wheel_link_br"/>
-    </joint>
-    <link name="wheel_link_br">
+      <parent link="${name}_caster_link_br"/>
+      <child link="${name}_wheel_link_br"/>
+    </joint>
+    <link name="${name}_wheel_link_br">
       <inertial>
         <mass value="${wheel_mass}"/>

Commit message: adjusted tinoBot xacro file which was (unexplicably) making the (kuka arm) IK fail

File: model/tinoBot.urdf.xacro (robot description, xacro)
@@ -122,4 +122,32 @@
         <material name="youBot/DarkGrey"/>
       </visual>
+      <visual>
+        <origin xyz="${caster_offset_x+wheel_offset_x} ${caster_offset_y+wheel_offset_y} ${caster_offset_z+wheel_offset_z}" rpy="0 0 0"/>
+        <geometry>
+          <sphere radius="${wheel_radius}"/>
+        </geometry>
+        <material name="youBot/Orange"/>
+      </visual>
+      <visual>
+        <origin xyz="${caster_offset_x+wheel_offset_x} ${-caster_offset_y+wheel_offset_y} ${caster_offset_z+wheel_offset_z}" rpy="0 0 0"/>
+        <geometry>
+          <sphere radius="${wheel_radius}"/>
+        </geometry>
+        <material name="youBot/Orange"/>
+      </visual>
+      <visual>
+        <origin xyz="${-caster_offset_x+wheel_offset_x} ${caster_offset_y+wheel_offset_y} ${caster_offset_z+wheel_offset_z}" rpy="0 0 0"/>
+        <geometry>
+          <sphere radius="${wheel_radius}"/>
+        </geometry>
+        <material name="youBot/Orange"/>
+      </visual>
+      <visual>
+        <origin xyz="${-caster_offset_x+wheel_offset_x} ${-caster_offset_y+wheel_offset_y} ${caster_offset_z+wheel_offset_z}" rpy="0 0 0"/>
+        <geometry>
+          <sphere radius="${wheel_radius}"/>
+        </geometry>
+        <material name="youBot/Orange"/>
+      </visual>
       <collision>
         <origin xyz="0 0 0" rpy="0 0 0"/>
@@ -130,39 +158,12 @@
       </collision>
     </link>
-    <!-- front left wheel -->
-    <joint name="${name}_caster_joint_fl" type="fixed"> <!-- type="continuous"> -->
-      <origin xyz="${caster_offset_x} ${caster_offset_y} ${caster_offset_z}" rpy="0 0 0"/>
-      <!-- <axis xyz="0 0 1"/>
-      <limit effort="${caster_joint_effort}" velocity="${caster_joint_velocity}"/>
-      <dynamics damping="${caster_joint_damping}" friction="${caster_joint_friction}"/>
-      <safety_controller k_velocity="${caster_joint_safety_k_velocity}"/> -->
+    <!-- <joint name="${name}_link_wheels" type="fixed">
+      <origin xyz="0 0 0" rpy="0 0 0"/>
+      <child link="${name}_wheels"/>
       <parent link="${name}_link"/>
-      <child link="${name}_caster_link_fl"/>
     </joint>
-    <link name="${name}_caster_link_fl">
-      <inertial>
-        <mass value="${caster_mass}"/>
-        <origin xyz="0 0 0"/>
-        <inertia ixx="0.012411765597" ixy="-0.000711733678" ixz="0.00050272983" iyy="0.015218160428" iyz="-0.000004273467" izz="0.011763977943"/>
-      </inertial>
-    </link>
-    <joint name="${name}_wheel_joint_fl" type="fixed"> <!-- type="continuous"> -->
-      <!-- <axis xyz="0 1 0"/>
-      <limit effort="${wheel_joint_effort}" velocity="${wheel_joint_velocity}"/>
-      <dynamics damping="${wheel_joint_damping}" friction="${wheel_joint_friction}"/>
-      <safety_controller k_velocity="${wheel_joint_safety_k_velocity}"/> -->
-      <origin xyz="${wheel_offset_x} ${wheel_offset_y} ${wheel_offset_z}" rpy="0 0 0"/>
-      <parent link="${name}_caster_link_fl"/>
-      <child link="${name}_wheel_link_fl"/>
-    </joint>
-    <link name="${name}_wheel_link_fl">
-      <inertial>
-        <mass value="${wheel_mass}"/>
-        <origin xyz="0 0 0"/>
-        <inertia ixx="0.012411765597" ixy="-0.000711733678" ixz="0.00050272983" iyy="0.015218160428" iyz="-0.000004273467" izz="0.011763977943"/>
-      </inertial>
+    <link name="${name}_wheels">
       <visual>
-        <origin xyz="0 0 0" rpy="0 0 0"/>
-        <!--<mesh filename="package://youbot_description/meshes/youbot_base/youbot_wheel.stl" />-->
+        <origin xyz="${caster_offset_x+wheel_offset_x} ${caster_offset_y+wheel_offset_y} ${caster_offset_z+wheel_offset_z}" rpy="0 0 0"/>
         <geometry>
           <sphere radius="${wheel_radius}"/>
@@ -170,156 +171,26 @@
         <material name="youBot/Orange"/>
       </visual>
-      <collision>
-        <origin xyz="0 0 0" rpy="${M_PI/2} 0 0"/>
+      <visual>
+        <origin xyz="${caster_offset_x+wheel_offset_x} ${-caster_offset_y+wheel_offset_y} ${caster_offset_z+wheel_offset_z}" rpy="0 0 0"/>
         <geometry>
-          <cylinder radius="${wheel_radius}" length="${wheel_radius}"/>
-        </geometry>
-      </collision>
-    </link>
-    <!-- front right wheel -->
-    <joint name="${name}_caster_joint_fr"  type="fixed"> <!-- type="continuous"> -->
-      <origin xyz="${caster_offset_x} ${-caster_offset_y} ${caster_offset_z}" rpy="0 0 0"/>
-      <!-- <axis xyz="0 0 1"/>
-      <limit effort="${caster_joint_effort}" velocity="${caster_joint_velocity}"/>
-      <dynamics damping="${caster_joint_damping}" friction="${caster_joint_friction}"/>
-      <safety_controller k_velocity="${caster_joint_safety_k_velocity}"/> -->
-      <parent link="${name}_link"/>
-      <child link="${name}_caster_link_fr"/>
-    </joint>
-    <link name="${name}_caster_link_fr">
-      <inertial>
-        <mass value="${caster_mass}"/>
-        <origin xyz="0 0 0"/>
-        <inertia ixx="0.012411765597" ixy="-0.000711733678" ixz="0.00050272983" iyy="0.015218160428" iyz="-0.000004273467" izz="0.011763977943"/>
-      </inertial>
-    </link>
-    <joint name="${name}_wheel_joint_fr"  type="fixed"> <!-- type="continuous"> -->
-      <!-- <axis xyz="0 1 0"/>
-      <limit effort="${wheel_joint_effort}" velocity="${wheel_joint_velocity}"/>
-      <dynamics damping="${wheel_joint_damping}" friction="${wheel_joint_friction}"/>
-      <safety_controller k_velocity="${wheel_joint_safety_k_velocity}"/> -->
-      <origin xyz="${wheel_offset_x} ${wheel_offset_y} ${wheel_offset_z}" rpy="0 0 0"/>
-      <parent link="${name}_caster_link_fr"/>
-      <child link="${name}_wheel_link_fr"/>
-    </joint>
-    <link name="${name}_wheel_link_fr">
-      <inertial>
-        <mass value="${wheel_mass}"/>
-        <origin xyz="0 0 0"/>
-        <inertia ixx="0.012411765597" ixy="-0.000711733678" ixz="0.00050272983" iyy="0.015218160428" iyz="-0.000004273467" izz="0.011763977943"/>
-      </inertial>
-      <visual>
-        <origin xyz="0 0 0" rpy="0 0 0"/>
-        <geometry>
-          <!--<mesh filename="package://youbot_description/meshes/youbot_base/youbot_wheel.stl" />-->
           <sphere radius="${wheel_radius}"/>
         </geometry>
         <material name="youBot/Orange"/>
       </visual>
-      <collision>
-        <origin xyz="0 0 0" rpy="${M_PI/2} 0 0"/>
+      <visual>
+        <origin xyz="${-caster_offset_x+wheel_offset_x} ${caster_offset_y+wheel_offset_y} ${caster_offset_z+wheel_offset_z}" rpy="0 0 0"/>
         <geometry>
-          <cylinder radius="${wheel_radius}" length="${wheel_radius}"/>
-        </geometry>
-      </collision>
-    </link>
-    <!-- back left wheel -->
-    <joint name="${name}_caster_joint_bl"  type="fixed"> <!-- type="continuous"> -->
-      <origin xyz="${-caster_offset_x} ${caster_offset_y} ${caster_offset_z}" rpy="0 0 0"/>
-      <!-- <axis xyz="0 0 1"/>
-      <limit effort="${caster_joint_effort}" velocity="${caster_joint_velocity}"/>
-      <dynamics damping="${caster_joint_damping}" friction="${caster_joint_friction}"/>
-      <safety_controller k_velocity="${caster_joint_safety_k_velocity}"/> -->
-      <parent link="${name}_link"/>
-      <child link="${name}_caster_link_bl"/>
-    </joint>
-    <link name="${name}_caster_link_bl">
-      <inertial>
-        <mass value="${caster_mass}"/>
-        <origin xyz="0 0 0"/>
-        <inertia ixx="0.012411765597" ixy="-0.000711733678" ixz="0.00050272983" iyy="0.015218160428" iyz="-0.000004273467" izz="0.011763977943"/>
-      </inertial>
-    </link>
-    <joint name="${name}_wheel_joint_bl"  type="fixed"> <!-- type="continuous"> -->
-      <!-- <axis xyz="0 1 0"/>
-      <limit effort="10" velocity="10"/>
-      <limit effort="${wheel_joint_effort}" velocity="${wheel_joint_velocity}"/>
-      <dynamics damping="${wheel_joint_damping}" friction="${wheel_joint_friction}"/>
-      <safety_controller k_velocity="${wheel_joint_safety_k_velocity}"/> -->
-      <origin xyz="${wheel_offset_x} ${wheel_offset_y} ${wheel_offset_z}" rpy="0 0 0"/>
-      <parent link="${name}_caster_link_bl"/>
-      <child link="${name}_wheel_link_bl"/>
-    </joint>
-    <link name="${name}_wheel_link_bl">
-      <inertial>
-        <mass value="${wheel_mass}"/>
-        <origin xyz="0 0 0"/>
-        <inertia ixx="0.012411765597" ixy="-0.000711733678" ixz="0.00050272983" iyy="0.015218160428" iyz="-0.000004273467" izz="0.011763977943"/>
-      </inertial>
-      <visual>
-        <origin xyz="0 0 0" rpy="0 0 0"/>
-        <geometry>
-          <!--<mesh filename="package://youbot_description/meshes/youbot_base/youbot_wheel.stl" />-->
           <sphere radius="${wheel_radius}"/>
         </geometry>
         <material name="youBot/Orange"/>
       </visual>
-      <collision>
-        <origin xyz="0 0 0" rpy="${M_PI/2} 0 0"/>
+      <visual>
+        <origin xyz="${-caster_offset_x+wheel_offset_x} ${-caster_offset_y+wheel_offset_y} ${caster_offset_z+wheel_offset_z}" rpy="0 0 0"/>
         <geometry>
-          <cylinder radius="${wheel_radius}" length="${wheel_radius}"/>
-        </geometry>
-      </collision>
-    </link>
-    <!-- back right wheel -->
-    <joint name="${name}_caster_joint_br" type="fixed"> <!-- type="continuous"> -->
-      <origin xyz="${-caster_offset_x} ${-caster_offset_y} ${caster_offset_z}" rpy="0 0 0"/>
-      <!-- <axis xyz="0 0 1"/>
-      <limit effort="${caster_joint_effort}" velocity="${caster_joint_velocity}"/>
-      <dynamics damping="${caster_joint_damping}" friction="${caster_joint_friction}"/>
-      <safety_controller k_velocity="${caster_joint_safety_k_velocity}"/> -->
-      <parent link="${name}_link"/>
-      <child link="${name}_caster_link_br"/>
-    </joint>
-    <link name="${name}_caster_link_br">
-      <inertial>
-        <mass value="${caster_mass}"/>
-        <origin xyz="0 0 0"/>
-        <inertia ixx="0.012411765597" ixy="-0.000711733678" ixz="0.00050272983" iyy="0.015218160428" iyz="-0.000004273467" izz="0.011763977943"/>
-      </inertial>
-    </link>
-    <joint name="${name}_wheel_joint_br" type="fixed"> <!-- type="continuous"> -->
-      <axis xyz="0 1 0"/>
-      <!-- <limit effort="${wheel_joint_effort}" velocity="${wheel_joint_velocity}"/>
-      <dynamics damping="${wheel_joint_damping}" friction="${wheel_joint_friction}"/>
-      <safety_controller k_velocity="${wheel_joint_safety_k_velocity}"/> -->
-      <origin xyz="${wheel_offset_x} ${wheel_offset_y} ${wheel_offset_z}" rpy="0 0 0"/>
-      <parent link="${name}_caster_link_br"/>
-      <child link="${name}_wheel_link_br"/>
-    </joint>
-    <link name="${name}_wheel_link_br">
-      <inertial>
-        <mass value="${wheel_mass}"/>
-        <origin xyz="0 0 0"/>
-        <inertia ixx="0.012411765597" ixy="-0.000711733678" ixz="0.00050272983" iyy="0.015218160428" iyz="-0.000004273467" izz="0.011763977943"/>
-      </inertial>
-      <visual>
-        <origin xyz="0 0 0" rpy="0 0 0"/>
-        <geometry>
-          <!--<mesh filename="package://youbot_description/meshes/youbot_base/youbot_wheel.stl" />-->
           <sphere radius="${wheel_radius}"/>
         </geometry>
         <material name="youBot/Orange"/>
       </visual>
-      <collision>
-        <origin xyz="0 0 0" rpy="${M_PI/2} 0 0"/>
-        <geometry>
-          <cylinder radius="${wheel_radius}" length="${wheel_radius}"/>
-        </geometry>
-      </collision>
-    </link>
-    <!-- extensions -->
-    <!-- <xacro:youbot_base_gazebo/> -->
-    <!-- <xacro:youbot_base_transmission/> -->
+    </link> -->
   </xacro:macro>
 </robot>

Commit message: slightly changed tinoBot xacro in order to simplify it

File: model/tinoBot.urdf.xacro (robot description, xacro)
@@ -1,9 +1,10 @@
 <?xml version="1.0"?>
-<robot xmlns:sensor="http://playerstage.sourceforge.net/gazebo/xmlschema/#sensor"
+<robot xmlns:xacro="http://ros.org/wiki/xacro">
+<!-- <robot xmlns:sensor="http://playerstage.sourceforge.net/gazebo/xmlschema/#sensor"
        xmlns:controller="http://playerstage.sourceforge.net/gazebo/xmlschema/#controller"
        xmlns:interface="http://playerstage.sourceforge.net/gazebo/xmlschema/#interface"
        xmlns:xacro="http://ros.org/wiki/xacro">
   <xacro:include filename="$(find youbot_description)/urdf/youbot_base/base.gazebo.xacro"/>
-  <xacro:include filename="$(find youbot_description)/urdf/youbot_base/base.transmission.xacro"/>
+  <xacro:include filename="$(find youbot_description)/urdf/youbot_base/base.transmission.xacro"/> -->
   <!-- simplified box collision geometry for base -->
   <property name="base_size_x" value="0.570"/>
@@ -61,12 +62,12 @@
     </joint>
     <link name="${name}_footprint_p2"/>
-    <joint name="${name}_base_p3_joint" type="continuous">
-      <origin xyz="0 0 0" rpy="0 0 0"/>
+    <joint name="${name}_base_p3_joint" type="revolute">
+      <origin xyz="0 0 0.1" rpy="0 0 0"/>
       <axis xyz="0 0 1"/>
-      <limit effort="${caster_joint_effort}" velocity="${caster_joint_velocity}"/>
+      <limit lower="-6.28" upper="6.28" effort="${caster_joint_effort}" velocity="${caster_joint_velocity}"/>
       <parent link="${name}_footprint_p2"/>
-      <child link="${name}_footprint"/>
+      <child link="${name}_link"/>
     </joint>
-    <link name="${name}_footprint">
+    <!-- <link name="${name}_footprint">
       <inertial>
         <mass value="0.1"/>
@@ -92,10 +93,9 @@
       <child link="${name}_link"/>
       <parent link="${name}_footprint"/>
-    </joint>
+    </joint> -->
     <joint name="${name}_ee_joint" type="fixed">
       <origin xyz="0 0 0.025" rpy="0 0 0"/>
-      <parent link="${name}_footprint"/>
+      <parent link="${name}_link"/>
       <child link="${name}_ee"/>
-      <!-- <child link="belt0_p"/> -->
     </joint>
     <!-- <link name="belt0_p"> -->
