Commit message: adjusted names in simple_factory to make it work with the simple, exemplary database

File: model/simple_factory.urdf.xacro (robot description, xacro)
@@ -34,34 +34,34 @@
   <xacro:model_table name="table0"
                     parent="simple_factory_anchor"
-                    length="1.0"
-                    width="1.30"
+                    length="0.5"
+                    width="1.0"
                     height="0.1"
                     plate_thickness="0.1">
-    <origin xyz="-3.0 0.65 0.1" rpy="0 0 0"/>
+    <origin xyz="-2.5 0.5 0.1" rpy="0 0 0"/>
   </xacro:model_table>
     <xacro:model_table name="table1"
                     parent="simple_factory_anchor"
-                    length="1.0"
-                    width="1.30"
+                    length="0.5"
+                    width="1.0"
                     height="0.1"
                     plate_thickness="0.1">
-    <origin xyz="2.0 0.65 0.1" rpy="0 0 0"/>
+    <origin xyz="2.0 0.5 0.1" rpy="0 0 0"/>
   </xacro:model_table>
   <!-- LEFT ARM 0 -->
   <xacro:kuka_lwr name="0_arm" parent="simple_factory_anchor">
-    <origin xyz="2.15 -0.5 0.1" rpy="0 0 ${M_PI*180.0/180}"/>
+    <origin xyz="2.0 -0.8 0.7" rpy="0 ${M_PI*90.0/180} ${M_PI*90.0/180}"/>
       <!-- rpy="${M_PI*80/180} ${M_PI*180.0/180} ${M_PI*0.0/180}"/> -->
   </xacro:kuka_lwr>
   <!-- LEFT SOFTHAND 0 -->
-  <xacro:soft_hand parent="0_arm_7_link" name="0_hand" left="false" withAdaptiveTransmission="true" useMimicTag="true">
+  <xacro:soft_hand parent="0_arm_7_link" name="0_right_hand" left="false" withAdaptiveTransmission="true" useMimicTag="true">
     <origin xyz="0 0 0" rpy="0 0 0"/>
   </xacro:soft_hand>
   <!-- RIGHT ARM 0 -->
   <xacro:kuka_lwr name="1_arm" parent="simple_factory_anchor">
-    <origin xyz="-2.15 0.5 0.10" rpy="0 0 ${M_PI*0.0/180}"/>
+    <origin xyz="-2.0 0.8 0.7" rpy="0 ${M_PI*90.0/180} ${M_PI*-90.0/180}"/>
       <!-- rpy="${M_PI*-80/180} ${M_PI*180.0/180} ${M_PI*0.0/180}"/> -->
   </xacro:kuka_lwr>
   <!-- RIGHT SOFTHAND 0 -->
-  <xacro:soft_hand parent="1_arm_7_link" name="1_hand" left="false" withAdaptiveTransmission="true" useMimicTag="true">
+  <xacro:soft_hand parent="1_arm_7_link" name="1_right_hand" left="false" withAdaptiveTransmission="true" useMimicTag="true">
     <origin xyz="0 0 0" rpy="0 0 0"/>
   </xacro:soft_hand>

File: model/tinoBot.urdf.xacro (robot description, xacro)
@@ -96,7 +96,9 @@
       <origin xyz="0 0 0.025" rpy="0 0 0"/>
       <parent link="${name}_footprint"/>
-      <child link="${name}_ee"/>
-    </joint>
-    <link name="${name}_ee">
+      <!-- <child link="${name}_ee"/> -->
+      <child link="belt0_p"/>
+    </joint>
+    <!-- <link name="${name}_ee"> -->
+    <link name="belt0_p">
       <visual>
         <origin xyz="0 0 0" rpy="0 0 0"/>

Commit message: adjusted simple_factory model and configuration

File: model/simple_factory.urdf.xacro (robot description, xacro)
@@ -29,16 +29,16 @@
        is the world frame). For more, see http://www.ros.org/wiki/xacro -->
   <link name="simple_factory_anchor" />
-  <!-- <xacro:robin name="tinoBot1" parent="simple_factory_anchor" px_lower_limit="-2" px_upper_limit="2" py_lower_limit="-1" py_upper_limit="1">
-    <origin xyz="0.0 0.0 0.0"/>
+  <xacro:robin name="tinoBot1" parent="simple_factory_anchor" px_lower_limit="-2" px_upper_limit="2" py_lower_limit="-1" py_upper_limit="1">
+    <origin xyz="0.0 0.0 -0.35"/>
   </xacro:robin>
-  <xacro:robin name="tinoBot2" parent="simple_factory_anchor" px_lower_limit="-2" px_upper_limit="2" py_lower_limit="-1" py_upper_limit="1">
+  <!-- <xacro:robin name="tinoBot2" parent="simple_factory_anchor" px_lower_limit="-2" px_upper_limit="2" py_lower_limit="-1" py_upper_limit="1">
     <origin xyz="0.0 1.0 0.0"/>
   </xacro:robin> -->
-  <xacro:tinoBot name="tinoBot1" parent="simple_factory_anchor">
+  <!-- <xacro:tinoBot name="tinoBot1" parent="simple_factory_anchor">
     <origin xyz="0 0 0.07"/>
-  </xacro:tinoBot>
+  </xacro:tinoBot> -->
   <!-- <xacro:tinoBot name="tinoBot2" parent="simple_factory_anchor" px_lower_limit="-2" px_upper_limit="2" py_lower_limit="-1" py_upper_limit="1">
-    <origin xyz="0 0.5 0.07"/> -->
-  </xacro:tinoBot>
+    <origin xyz="0 0.5 0.07"/>
+  </xacro:tinoBot> -->
   <!-- TABLES -->
   <xacro:model_table name="table0"
@@ -46,5 +46,5 @@
                     length="0.5"
                     width="1.0"
-                    height="0.1"
+                    height="0.45"
                     plate_thickness="0.1">
     <origin xyz="-2.5 0.5 0.1" rpy="0 0 0"/>
@@ -54,5 +54,5 @@
                     length="0.5"
                     width="1.0"
-                    height="0.1"
+                    height="0.45"
                     plate_thickness="0.1">
     <origin xyz="2.0 0.5 0.1" rpy="0 0 0"/>
@@ -76,3 +76,33 @@
     <origin xyz="0 0 0" rpy="0 0 0"/>
   </xacro:soft_hand>
+  <!-- a collision column in the scene -->
+  <joint name="simple_factory_column_1_joint" type="fixed">
+    <origin xyz="-1.5 0.8 0.0" rpy="0 0 0" />
+    <parent link="simple_factory_anchor" />
+    <child link="simple_factory_column_1_link" />
+  </joint>
+  <link name="simple_factory_column_1_link">
+    <collision>
+      <origin xyz="0.0 0.0 0.0" rpy="0 0 0" />
+      <geometry>
+         <cylinder length="1.4" radius="0.35" />
+         <!-- <box size="1.0 0.3 1.4"/> -->
+      </geometry>
+    </collision>
+  </link>
+  <!-- a collision column in the scene -->
+  <joint name="simple_factory_column_2_joint" type="fixed">
+    <origin xyz="1.5 -0.8 0.0" rpy="0 0 0" />
+    <parent link="simple_factory_anchor" />
+    <child link="simple_factory_column_2_link" />
+  </joint>
+  <link name="simple_factory_column_2_link">
+    <collision>
+      <origin xyz="0.0 0.0 0.0" rpy="0 0 0" />
+      <geometry>
+         <cylinder length="1.4" radius="0.35" />
+         <!-- <box size="1.0 0.3 1.4"/> -->
+      </geometry>
+    </collision>
+  </link>
 </robot>
