Commit message: trying out robin robots instead of youbots

File: model/bi_tino_simple_factory.urdf.xacro (robot description, xacro)
@@ -13,4 +13,5 @@
   <xacro:include filename="$(find soft_hand_description)/model/soft_hand.urdf.xacro"/>
   <xacro:include filename="$(find dual_manipulation_shared)/model/tinoBot.urdf.xacro" />
+  <xacro:include filename="$(find dual_manipulation_shared)/model/robin.urdf.xacro" />
   <!-- controller manager -->
   <!-- <xacro:include filename="$(find youbot_description)/controller/ros_controller.urdf.xacro" /> -->
@@ -28,10 +29,16 @@
        is the world frame). For more, see http://www.ros.org/wiki/xacro -->
   <link name="bi_tino_simple_factory_anchor" />
-  <xacro:tinoBot name="tinoBot1" parent="bi_tino_simple_factory_anchor" px_lower_limit="-2" px_upper_limit="2" py_lower_limit="-1" py_upper_limit="1">
+  <xacro:robin name="tinoBot1" parent="bi_tino_simple_factory_anchor" px_lower_limit="-2" px_upper_limit="2" py_lower_limit="-1" py_upper_limit="1">
+    <origin xyz="0.0 -0.5 -0.7"/>
+  </xacro:robin>
+  <xacro:robin name="tinoBot2" parent="bi_tino_simple_factory_anchor" px_lower_limit="-2" px_upper_limit="2" py_lower_limit="-1" py_upper_limit="1">
+    <origin xyz="0.0 0.5 -0.7"/>
+  </xacro:robin>
+  <!-- <xacro:tinoBot name="tinoBot1" parent="bi_tino_simple_factory_anchor" px_lower_limit="-2" px_upper_limit="2" py_lower_limit="-1" py_upper_limit="1">
     <origin xyz="0 -0.5 0.07"/>
-  </xacro:tinoBot>
-  <xacro:tinoBot name="tinoBot2" parent="bi_tino_simple_factory_anchor" px_lower_limit="-2" px_upper_limit="2" py_lower_limit="-1" py_upper_limit="1">
+  </xacro:tinoBot> -->
+  <!-- <xacro:tinoBot name="tinoBot2" parent="bi_tino_simple_factory_anchor" px_lower_limit="-2" px_upper_limit="2" py_lower_limit="-1" py_upper_limit="1">
     <origin xyz="0 0.5 0.07"/>
-  </xacro:tinoBot>
+  </xacro:tinoBot> -->
   <!-- TABLES -->
   <xacro:model_table name="table0"

File: model/simple_factory.urdf.xacro (robot description, xacro)
@@ -13,4 +13,5 @@
   <xacro:include filename="$(find soft_hand_description)/model/soft_hand.urdf.xacro"/>
   <xacro:include filename="$(find dual_manipulation_shared)/model/tinoBot.urdf.xacro" />
+  <xacro:include filename="$(find dual_manipulation_shared)/model/robin.urdf.xacro" />
   <!-- controller manager -->
   <!-- <xacro:include filename="$(find youbot_description)/controller/ros_controller.urdf.xacro" /> -->
@@ -28,6 +29,15 @@
        is the world frame). For more, see http://www.ros.org/wiki/xacro -->
   <link name="simple_factory_anchor" />
-  <xacro:tinoBot name="tinoBot" parent="simple_factory_anchor">
+  <!-- <xacro:robin name="tinoBot1" parent="simple_factory_anchor" px_lower_limit="-2" px_upper_limit="2" py_lower_limit="-1" py_upper_limit="1">
+    <origin xyz="0.0 0.0 0.0"/>
+  </xacro:robin>
+  <xacro:robin name="tinoBot2" parent="simple_factory_anchor" px_lower_limit="-2" px_upper_limit="2" py_lower_limit="-1" py_upper_limit="1">
+    <origin xyz="0.0 1.0 0.0"/>
+  </xacro:robin> -->
+  <xacro:tinoBot name="tinoBot1" parent="simple_factory_anchor">
     <origin xyz="0 0 0.07"/>
+  </xacro:tinoBot>
+  <!-- <xacro:tinoBot name="tinoBot2" parent="simple_factory_anchor" px_lower_limit="-2" px_upper_limit="2" py_lower_limit="-1" py_upper_limit="1">
+    <origin xyz="0 0.5 0.07"/> -->
   </xacro:tinoBot>
   <!-- TABLES -->

Commit message: added columns in the collision scene of bi_tino robot

File: model/bi_tino_simple_factory.urdf.xacro (robot description, xacro)
@@ -28,10 +28,18 @@
        the origin block defines where the component is w.r.t its parent (in this case the parent
        is the world frame). For more, see http://www.ros.org/wiki/xacro -->
+  <property name="tinoBot1_y_center" value="-0.3"/>
+  <!-- <property name="tinoBot1_y_ll" value="-1-(${tinoBot1_y_center})"/>
+  <property name="tinoBot1_y_ul" value="1-(${tinoBot1_y_center})"/> -->
+  <property name="tinoBot2_y_center" value="0.3"/>
+  <!-- <property name="tinoBot1_y_ll" value="-1-(${tinoBot2_y_center})"/>
+  <property name="tinoBot1_y_ul" value="1-(${tinoBot2_y_center})"/> -->
   <link name="bi_tino_simple_factory_anchor" />
   <xacro:robin name="tinoBot1" parent="bi_tino_simple_factory_anchor" px_lower_limit="-2" px_upper_limit="2" py_lower_limit="-1" py_upper_limit="1">
-    <origin xyz="0.0 -0.5 -0.7"/>
+    <!-- py_lower_limit="${-1-tinoBot1_y_center}" py_upper_limit="${1-tinoBot1_y_center}"> -->
+    <origin xyz="0.0 ${tinoBot1_y_center} -0.35"/>
   </xacro:robin>
   <xacro:robin name="tinoBot2" parent="bi_tino_simple_factory_anchor" px_lower_limit="-2" px_upper_limit="2" py_lower_limit="-1" py_upper_limit="1">
-    <origin xyz="0.0 0.5 -0.7"/>
+    <!-- py_lower_limit="${-1-tinoBot2_y_center}" py_upper_limit="${1-tinoBot2_y_center}"> -->
+    <origin xyz="0.0 ${tinoBot2_y_center} -0.35"/>
   </xacro:robin>
   <!-- <xacro:tinoBot name="tinoBot1" parent="bi_tino_simple_factory_anchor" px_lower_limit="-2" px_upper_limit="2" py_lower_limit="-1" py_upper_limit="1">
@@ -46,5 +54,5 @@
                     length="0.5"
                     width="1.0"
-                    height="0.1"
+                    height="0.45"
                     plate_thickness="0.1">
     <origin xyz="-2.5 0.5 0.1" rpy="0 0 0"/>
@@ -54,5 +62,5 @@
                     length="0.5"
                     width="1.0"
-                    height="0.1"
+                    height="0.45"
                     plate_thickness="0.1">
     <origin xyz="2.0 0.5 0.1" rpy="0 0 0"/>
@@ -76,3 +84,61 @@
     <origin xyz="0 0 0" rpy="0 0 0"/>
   </xacro:soft_hand>
+  <!-- a collision column in the scene -->
+  <joint name="bi_tino_column_1_joint" type="fixed">
+    <origin xyz="-1.5 0.8 0.0" rpy="0 0 0" />
+    <parent link="bi_tino_simple_factory_anchor" />
+    <child link="bi_tino_column_1_link" />
+  </joint>
+  <link name="bi_tino_column_1_link">
+    <collision>
+      <origin xyz="0.0 0.0 0.0" rpy="0 0 0" />
+      <geometry>
+         <cylinder length="1.4" radius="0.35" />
+         <!-- <box size="1.0 0.3 1.4"/> -->
+      </geometry>
+    </collision>
+  </link>
+  <!-- a collision column in the scene -->
+  <joint name="bi_tino_column_2_joint" type="fixed">
+    <origin xyz="1.5 -0.8 0.0" rpy="0 0 0" />
+    <parent link="bi_tino_simple_factory_anchor" />
+    <child link="bi_tino_column_2_link" />
+  </joint>
+  <link name="bi_tino_column_2_link">
+    <collision>
+      <origin xyz="0.0 0.0 0.0" rpy="0 0 0" />
+      <geometry>
+         <cylinder length="1.4" radius="0.35" />
+         <!-- <box size="1.0 0.3 1.4"/> -->
+      </geometry>
+    </collision>
+  </link>
+  <!-- a collision box in the scene -->
+  <!-- <joint name="bi_tino_box_1_joint" type="fixed">
+    <origin xyz="0.0 -0.5 0.0" rpy="0 0 0" />
+    <parent link="bi_tino_simple_factory_anchor" />
+    <child link="bi_tino_box_1_link" />
+  </joint>
+  <link name="bi_tino_box_1_link">
+    <collision>
+      <origin xyz="0.0 0.0 0.0" rpy="0 0 0" />
+      <geometry>
+         <box size="1.5 0.99 1.4"/>
+      </geometry>
+    </collision>
+  </link> -->
+  <!-- a collision box in the scene -->
+  <!-- <joint name="bi_tino_box_2_joint" type="fixed">
+    <origin xyz="0.0 0.5 0.0" rpy="0 0 0" />
+    <parent link="bi_tino_simple_factory_anchor" />
+    <child link="bi_tino_box_2_link" />
+  </joint>
+  <link name="bi_tino_box_2_link">
+    <collision>
+      <origin xyz="0.0 0.0 0.0" rpy="0 0 0" />
+      <geometry>
+         <box size="1.5 0.99 1.4"/>
+      </geometry>
+    </collision>
+  </link> -->
 </robot>

Commit message: adjusted some parameters in bi_tino_simple_factory

File: model/bi_tino_simple_factory.urdf.xacro (robot description, xacro)
@@ -85,5 +85,5 @@
   </xacro:soft_hand>
   <!-- a collision column in the scene -->
-  <joint name="bi_tino_column_1_joint" type="fixed">
+  <!-- <joint name="bi_tino_column_1_joint" type="fixed">
     <origin xyz="-1.5 0.8 0.0" rpy="0 0 0" />
     <parent link="bi_tino_simple_factory_anchor" />
@@ -95,10 +95,10 @@
       <geometry>
          <cylinder length="1.4" radius="0.35" />
-         <!-- <box size="1.0 0.3 1.4"/> -->
       </geometry>
     </collision>
-  </link>
+  </link> -->
+         <!-- <box size="1.0 0.3 1.4"/> -->
   <!-- a collision column in the scene -->
-  <joint name="bi_tino_column_2_joint" type="fixed">
+  <!-- <joint name="bi_tino_column_2_joint" type="fixed">
     <origin xyz="1.5 -0.8 0.0" rpy="0 0 0" />
     <parent link="bi_tino_simple_factory_anchor" />
@@ -110,8 +110,8 @@
       <geometry>
          <cylinder length="1.4" radius="0.35" />
-         <!-- <box size="1.0 0.3 1.4"/> -->
       </geometry>
     </collision>
-  </link>
+  </link> -->
+         <!-- <box size="1.0 0.3 1.4"/> -->
   <!-- a collision box in the scene -->
   <!-- <joint name="bi_tino_box_1_joint" type="fixed">

Commit message: xacro modified previously

File: model/bi_tino_simple_factory.urdf.xacro (robot description, xacro)
@@ -28,10 +28,10 @@
        the origin block defines where the component is w.r.t its parent (in this case the parent
        is the world frame). For more, see http://www.ros.org/wiki/xacro -->
-  <property name="tinoBot1_y_center" value="-0.3"/>
-  <!-- <property name="tinoBot1_y_ll" value="-1-(${tinoBot1_y_center})"/>
-  <property name="tinoBot1_y_ul" value="1-(${tinoBot1_y_center})"/> -->
-  <property name="tinoBot2_y_center" value="0.3"/>
-  <!-- <property name="tinoBot1_y_ll" value="-1-(${tinoBot2_y_center})"/>
-  <property name="tinoBot1_y_ul" value="1-(${tinoBot2_y_center})"/> -->
+  <xacro:property name="tinoBot1_y_center" value="-0.3"/>
+  <!-- <xacro:property name="tinoBot1_y_ll" value="-1-(${tinoBot1_y_center})"/>
+  <xacro:property name="tinoBot1_y_ul" value="1-(${tinoBot1_y_center})"/> -->
+  <xacro:property name="tinoBot2_y_center" value="0.3"/>
+  <!-- <xacro:property name="tinoBot1_y_ll" value="-1-(${tinoBot2_y_center})"/>
+  <xacro:property name="tinoBot1_y_ul" value="1-(${tinoBot2_y_center})"/> -->
   <link name="bi_tino_simple_factory_anchor" />
   <xacro:robin name="tinoBot1" parent="bi_tino_simple_factory_anchor" px_lower_limit="-2" px_upper_limit="2" py_lower_limit="-1" py_upper_limit="1">

File: model/conveyor_belt.urdf.xacro (robot description, xacro)
@@ -16,5 +16,5 @@
 <xacro:macro name="model_belt" params="parent name *origin length width height leg_length plate_thickness">
     <joint name="${parent}_${name}_base_joint" type="fixed">
-        <insert_block name="origin"/>
+        <xacro:insert_block name="origin"/>
         <parent link="${parent}"/>
         <child link="${name}_plate_link"/>
@@ -22,5 +22,5 @@
     <link name="${name}_plate_link">
         <inertial>
-            <insert_block name="negligible_inertia"/>
+            <xacro:insert_block name="negligible_inertia"/>
         </inertial>
         <visual>
@@ -45,5 +45,5 @@
     <link name="${name}_link1">
         <inertial>
-            <insert_block name="negligible_inertia"/>
+            <xacro:insert_block name="negligible_inertia"/>
         </inertial>
         <visual>
@@ -69,5 +69,5 @@
     <link name="${name}_cylinder_leg1">
         <inertial>
-            <insert_block name="negligible_inertia"/>
+            <xacro:insert_block name="negligible_inertia"/>
         </inertial>
         <visual>
@@ -93,5 +93,5 @@
     <link name="${name}_cylinder_leg2">
         <inertial>
-            <insert_block name="negligible_inertia"/>
+            <xacro:insert_block name="negligible_inertia"/>
         </inertial>
         <visual>
@@ -118,5 +118,5 @@
     <link name="${name}_link2">
         <inertial>
-            <insert_block name="negligible_inertia"/>
+            <xacro:insert_block name="negligible_inertia"/>
         </inertial>
         <visual>
@@ -142,5 +142,5 @@
     <link name="${name}_cylinder_leg3">
         <inertial>
-            <insert_block name="negligible_inertia"/>
+            <xacro:insert_block name="negligible_inertia"/>
         </inertial>
         <visual>
@@ -166,5 +166,5 @@
     <link name="${name}_cylinder_leg4">
         <inertial>
-            <insert_block name="negligible_inertia"/>
+            <xacro:insert_block name="negligible_inertia"/>
         </inertial>
         <visual>
@@ -196,5 +196,5 @@
     <link name="${name}_p_1">
         <inertial>
-            <insert_block name="negligible_inertia"/>
+            <xacro:insert_block name="negligible_inertia"/>
         </inertial>
     </link>
@@ -209,5 +209,5 @@
     <link name="${name}_p">
         <inertial>
-            <insert_block name="negligible_inertia"/>
+            <xacro:insert_block name="negligible_inertia"/>
         </inertial>
         <visual>

File: model/robin.urdf.xacro (robot description, xacro)
@@ -2,8 +2,8 @@
 <!-- modified version of omnirob_robin_base from github.com/robinJKU/omnirob_robin -->
 <robot xmlns:xacro="http://www.ros.org/wiki/xacro">
-   <property name="px_lower_limit_def" value="-2"/>
-   <property name="px_upper_limit_def" value="2"/>
-   <property name="py_lower_limit_def" value="-1"/>
-   <property name="py_upper_limit_def" value="1"/>
+   <xacro:property name="px_lower_limit_def" value="-2"/>
+   <xacro:property name="px_upper_limit_def" value="2"/>
+   <xacro:property name="py_lower_limit_def" value="-1"/>
+   <xacro:property name="py_upper_limit_def" value="1"/>
    <xacro:macro name="robin" params="parent name *origin px_lower_limit:=${px_lower_limit_def} px_upper_limit:=${px_upper_limit_def} py_lower_limit:=${py_lower_limit_def} py_upper_limit:=${py_upper_limit_def}">
       <!-- <link name="world" />
@@ -20,5 +20,5 @@
       </link> -->
       <joint name="${name}_base_p1_joint" type="prismatic">
-         <insert_block name="origin"/>
+         <xacro:insert_block name="origin"/>
          <axis xyz="1 0 0" />
          <dynamics damping="0.0" friction="0.0" />

File: model/shelf.urdf.xacro (robot description, xacro)
@@ -16,5 +16,5 @@
 <xacro:macro name="model_shelf" params="parent name *origin length width height plate_thickness color">
     <joint name="${parent}_${name}_base_joint" type="fixed">
-        <insert_block name="origin"/>
+        <xacro:insert_block name="origin"/>
         <parent link="${parent}"/>
         <child link="${name}_plate_link"/>
@@ -22,5 +22,5 @@
     <link name="${name}_plate_link">
         <inertial>
-            <insert_block name="negligible_inertia"/>
+            <xacro:insert_block name="negligible_inertia"/>
         </inertial>
         <visual>

File: model/tinoBot.urdf.xacro (robot description, xacro)
@@ -8,37 +8,37 @@
   <xacro:include filename="$(find youbot_description)/urdf/youbot_base/base.transmission.xacro"/> -->
   <!-- simplified box collision geometry for base -->
-  <property name="base_size_x" value="0.570"/>
-  <property name="base_size_y" value="0.360"/>
-  <property name="base_size_z" value="0.100"/>
-  <property name="base_mass" value="22.0"/>
-  <property name="caster_offset_x" value="0.228"/>
-  <property name="caster_offset_y" value="0.158"/>
-  <property name="caster_offset_z" value="-0.034"/>
-  <property name="caster_mass" value="0.1"/>
-  <property name="wheel_offset_x" value="0.0"/>
-  <property name="wheel_offset_y" value="0.0"/>
-  <property name="wheel_offset_z" value="0.0"/>
-  <property name="wheel_mass" value="1.4"/>
-  <property name="wheel_radius" value="0.0475"/>
-  <property name="wheel_length" value="0.005"/>
-  <property name="caster_joint_damping" value="1.0"/>
-  <property name="caster_joint_friction" value="1.0"/>
-  <property name="caster_joint_effort" value="30"/>
-  <property name="caster_joint_velocity" value="10"/>
-  <property name="caster_joint_safety_k_velocity" value="10.0"/>
-  <property name="wheel_joint_damping" value="1.0"/>
-  <property name="wheel_joint_friction" value="1.0"/>
-  <property name="wheel_joint_effort" value="30"/>
-  <property name="wheel_joint_velocity" value="10"/>
-  <property name="wheel_joint_safety_k_velocity" value="10.0"/>
-  <property name="p_joint_effort" value="30"/>
-  <property name="p_joint_velocity" value="10"/>
-  <property name="px_lower_limit_def" value="-2"/>
-  <property name="px_upper_limit_def" value="2"/>
-  <property name="py_lower_limit_def" value="-1"/>
-  <property name="py_upper_limit_def" value="1"/>
+  <xacro:property name="base_size_x" value="0.570"/>
+  <xacro:property name="base_size_y" value="0.360"/>
+  <xacro:property name="base_size_z" value="0.100"/>
+  <xacro:property name="base_mass" value="22.0"/>
+  <xacro:property name="caster_offset_x" value="0.228"/>
+  <xacro:property name="caster_offset_y" value="0.158"/>
+  <xacro:property name="caster_offset_z" value="-0.034"/>
+  <xacro:property name="caster_mass" value="0.1"/>
+  <xacro:property name="wheel_offset_x" value="0.0"/>
+  <xacro:property name="wheel_offset_y" value="0.0"/>
+  <xacro:property name="wheel_offset_z" value="0.0"/>
+  <xacro:property name="wheel_mass" value="1.4"/>
+  <xacro:property name="wheel_radius" value="0.0475"/>
+  <xacro:property name="wheel_length" value="0.005"/>
+  <xacro:property name="caster_joint_damping" value="1.0"/>
+  <xacro:property name="caster_joint_friction" value="1.0"/>
+  <xacro:property name="caster_joint_effort" value="30"/>
+  <xacro:property name="caster_joint_velocity" value="10"/>
+  <xacro:property name="caster_joint_safety_k_velocity" value="10.0"/>
+  <xacro:property name="wheel_joint_damping" value="1.0"/>
+  <xacro:property name="wheel_joint_friction" value="1.0"/>
+  <xacro:property name="wheel_joint_effort" value="30"/>
+  <xacro:property name="wheel_joint_velocity" value="10"/>
+  <xacro:property name="wheel_joint_safety_k_velocity" value="10.0"/>
+  <xacro:property name="p_joint_effort" value="30"/>
+  <xacro:property name="p_joint_velocity" value="10"/>
+  <xacro:property name="px_lower_limit_def" value="-2"/>
+  <xacro:property name="px_upper_limit_def" value="2"/>
+  <xacro:property name="py_lower_limit_def" value="-1"/>
+  <xacro:property name="py_upper_limit_def" value="1"/>
   <xacro:macro name="tinoBot" params="parent name *origin px_lower_limit:=${px_lower_limit_def} px_upper_limit:=${px_upper_limit_def} py_lower_limit:=${py_lower_limit_def} py_upper_limit:=${py_upper_limit_def}">
     <!-- <joint name="${name}_base_joint" type="fixed">
-      <insert_block name="origin"/>
+      <xacro:insert_block name="origin"/>
       <origin xyz="0 0 0" rpy="0 0 0"/>
       <parent link="${parent}"/>
@@ -46,5 +46,5 @@
     </joint> -->
     <joint name="${name}_base_p1_joint" type="prismatic">
-      <insert_block name="origin"/>
+      <xacro:insert_block name="origin"/>
       <origin xyz="0 0 0" rpy="0 0 0"/>
       <axis xyz="1 0 0"/>

File: model/tinoBot_bad_wheels.urdf.xacro (robot description, xacro)
@@ -7,37 +7,37 @@
   <xacro:include filename="$(find youbot_description)/urdf/youbot_base/base.transmission.xacro"/>
   <!-- simplified box collision geometry for base -->
-  <property name="base_size_x" value="0.570"/>
-  <property name="base_size_y" value="0.360"/>
-  <property name="base_size_z" value="0.100"/>
-  <property name="base_mass" value="22.0"/>
-  <property name="caster_offset_x" value="0.228"/>
-  <property name="caster_offset_y" value="0.158"/>
-  <property name="caster_offset_z" value="-0.034"/>
-  <property name="caster_mass" value="0.1"/>
-  <property name="wheel_offset_x" value="0.0"/>
-  <property name="wheel_offset_y" value="0.0"/>
-  <property name="wheel_offset_z" value="0.0"/>
-  <property name="wheel_mass" value="1.4"/>
-  <property name="wheel_radius" value="0.0475"/>
-  <property name="wheel_length" value="0.005"/>
-  <property name="caster_joint_damping" value="1.0"/>
-  <property name="caster_joint_friction" value="1.0"/>
-  <property name="caster_joint_effort" value="30"/>
-  <property name="caster_joint_velocity" value="10"/>
-  <property name="caster_joint_safety_k_velocity" value="10.0"/>
-  <property name="wheel_joint_damping" value="1.0"/>
-  <property name="wheel_joint_friction" value="1.0"/>
-  <property name="wheel_joint_effort" value="30"/>
-  <property name="wheel_joint_velocity" value="10"/>
-  <property name="wheel_joint_safety_k_velocity" value="10.0"/>
-  <property name="p_joint_effort" value="30"/>
-  <property name="p_joint_velocity" value="10"/>
-  <property name="px_lower_limit_def" value="-2"/>
-  <property name="px_upper_limit_def" value="2"/>
-  <property name="py_lower_limit_def" value="-1"/>
-  <property name="py_upper_limit_def" value="1"/>
+  <xacro:property name="base_size_x" value="0.570"/>
+  <xacro:property name="base_size_y" value="0.360"/>
+  <xacro:property name="base_size_z" value="0.100"/>
+  <xacro:property name="base_mass" value="22.0"/>
+  <xacro:property name="caster_offset_x" value="0.228"/>
+  <xacro:property name="caster_offset_y" value="0.158"/>
+  <xacro:property name="caster_offset_z" value="-0.034"/>
+  <xacro:property name="caster_mass" value="0.1"/>
+  <xacro:property name="wheel_offset_x" value="0.0"/>
+  <xacro:property name="wheel_offset_y" value="0.0"/>
+  <xacro:property name="wheel_offset_z" value="0.0"/>
+  <xacro:property name="wheel_mass" value="1.4"/>
+  <xacro:property name="wheel_radius" value="0.0475"/>
+  <xacro:property name="wheel_length" value="0.005"/>
+  <xacro:property name="caster_joint_damping" value="1.0"/>
+  <xacro:property name="caster_joint_friction" value="1.0"/>
+  <xacro:property name="caster_joint_effort" value="30"/>
+  <xacro:property name="caster_joint_velocity" value="10"/>
+  <xacro:property name="caster_joint_safety_k_velocity" value="10.0"/>
+  <xacro:property name="wheel_joint_damping" value="1.0"/>
+  <xacro:property name="wheel_joint_friction" value="1.0"/>
+  <xacro:property name="wheel_joint_effort" value="30"/>
+  <xacro:property name="wheel_joint_velocity" value="10"/>
+  <xacro:property name="wheel_joint_safety_k_velocity" value="10.0"/>
+  <xacro:property name="p_joint_effort" value="30"/>
+  <xacro:property name="p_joint_velocity" value="10"/>
+  <xacro:property name="px_lower_limit_def" value="-2"/>
+  <xacro:property name="px_upper_limit_def" value="2"/>
+  <xacro:property name="py_lower_limit_def" value="-1"/>
+  <xacro:property name="py_upper_limit_def" value="1"/>
   <xacro:macro name="tinoBot" params="parent name *origin px_lower_limit:=${px_lower_limit_def} px_upper_limit:=${px_upper_limit_def} py_lower_limit:=${py_lower_limit_def} py_upper_limit:=${py_upper_limit_def}">
     <!-- <joint name="${name}_base_joint" type="fixed">
-      <insert_block name="origin"/>
+      <xacro:insert_block name="origin"/>
       <origin xyz="0 0 0" rpy="0 0 0"/>
       <parent link="${parent}"/>
@@ -45,5 +45,5 @@
     </joint> -->
     <joint name="${name}_base_p1_joint" type="prismatic">
-      <insert_block name="origin"/>
+      <xacro:insert_block name="origin"/>
       <origin xyz="0 0 0" rpy="0 0 0"/>
       <axis xyz="1 0 0"/>
